Commit message: Readme de ejercicio5 con gif

File: src/primer_paquete_2026/ejercicio5/robot_description/dp/dp.xacro (robot description, xacro)
@@ -92,7 +92,5 @@
     <child link="link1" />
     <origin xyz="0 0 ${height0+width1/2.0}" rpy="0 0 0" />
-    <axis xyz="0 0 1">
-      <initial_position>$(arg q1_ini)</initial_position>
-    </axis>
+    <axis xyz="0 0 1" />
     <limit effort="$(arg tau1_max)" lower="$(arg q1_min)" upper="$(arg q1_max)"
       velocity="$(arg qp1_max)" />
@@ -104,7 +102,5 @@
     <child link="link2" />
     <origin xyz="${a1} 0 ${-width1}" rpy="0 0 0" />
-    <axis xyz="0 0 1">
-      <initial_position>$(arg q2_ini)</initial_position>
-    </axis>
+    <axis xyz="0 0 1" />
     <limit effort="$(arg tau2_max)" lower="$(arg q2_min)" upper="$(arg q2_max)"
       velocity="$(arg qp2_max)" />
